Commit message: added branching computations

File: third_party/urdfs/panda4dofBranching.urdf (robot description, URDF)
Before this commit: robot panda, 5 links, 4 joints
Links:
- added link panda_link5, mass 2.38; collision mesh filename=link3.stl; visual mesh filename=link3.stl
- added link panda_link6, mass 2.38; collision mesh filename=link4.stl; visual mesh filename=link4.stl
Joints:
- added joint panda_joint5: type revolute, parent panda_link2, child panda_link5, origin xyz=0 -0.316 0 rpy=1.57079632679 0 0, axis 0 0 1, limit lower=-2.9671 upper=2.9671 effort=87 velocity=2.1750
- added joint panda_joint6: type revolute, parent panda_link5, child panda_link6, origin xyz=0.0825 0 0 rpy=1.57079632679 0 0, axis 0 0 1, limit lower=-3.1416 upper=0.0 effort=87 velocity=2.1750
